File: PowerManagementBoard/PowerManagementSchem.brd (EAGLE design)
At the start: 165.1 x 106.7 mm, 92 parts, among them J1 D15S24A4GV00LF, J8 182-037-213R531, J9 182-025-213R531, U1 VX7805-500, U2 PYB20-Q24-S5, U3 PYB30-Q48-S5, U4 PYB30-Q48-S12, U5 3V3REG, U6 INA4180-SPLIT, U7 INA4180-SPLIT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

Commit message: Did some stuff
Routing:
- net 12V-CAM: track 0.00 -> 21.1 mm
- net 12V-STA: track 0.00 -> 19.8 mm
- net 5V-ACT-CAM: track 0.00 -> 7.12 mm
- net 5V-ACT-TX: track 0.00 -> 6.98 mm
- net 5V-DIG-TX: track 0.00 -> 6.92 mm
- net 5V-DIG-CAM: track 0.00 -> 5.76 mm
- net 5V-DIG-STA: track 0.00 -> 4.00 mm
- net 5V-DIG-LASER: track 0.00 -> 3.95 mm
- net 5V-ACT-STA: track 0.00 -> 3.90 mm
- net 5V-ACT-LASER: track 0.00 -> 3.80 mm
- net 5V-DIG-MAG: track 0.00 -> 3.52 mm
- net 5V-ACT-MAG: track 0.00 -> 2.20 mm
Other:
- board text added: "To make this work, I think we need to use 32 mil trace for our 2A lines. I know it will lead to hot traces, but it only runs for 3 minutes. Some calculators say only 10C rise for 2.2A load"
Changed lines of the file:
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@@
 -Route big power traces, route traces that go near mosfets
 -Now, place minor components like small vregs in the free space</text>
+<text x="173.99" y="46.99" size="1.9304" layer="48">To make this work, I think we need to use 32 mil
+trace for our 2A lines. I know it will lead to hot
+traces, but it only runs for 3 minutes. Some
+calculators say only 10C rise for 2.2A load</text>
 </plain>
 <attributes>
@@
 </element>
 <element name="U$1" library="usbMotorDriverParts" package="DPAK" package3d_urn="urn:adsk.eagle:package:38459/1" value="PMOSFET" x="72.39" y="-125.73" smashed="yes">
-<attribute name="NAME" x="69.85" y="-214.63" size="0.6096" layer="25" font="vector" ratio="20" rot="R90" align="bottom-center"/>
 <attribute name="VALUE" x="76.2" y="-125.73" size="0.6096" layer="27" font="vector" ratio="20" rot="R90" align="top-center"/>
 </element>
@@
 </element>
 <element name="U$6" library="usbMotorDriverParts" package="DPAK" package3d_urn="urn:adsk.eagle:package:38459/1" value="PMOSFET" x="43.18" y="-129.54" smashed="yes">
-<attribute name="NAME" x="34.29" y="-232.41" size="0.6096" layer="25" font="vector" ratio="20" rot="R90" align="bottom-center"/>
 <attribute name="VALUE" x="46.99" y="-129.54" size="0.6096" layer="27" font="vector" ratio="20" rot="R90" align="top-center"/>
 </element>
@@
 </element>
 <element name="U$16" library="usbMotorDriverParts" package="DPAK" package3d_urn="urn:adsk.eagle:package:38459/1" value="PMOSFET" x="72.39" y="-100.33" smashed="yes">
-<attribute name="NAME" x="88.9" y="-247.65" size="0.6096" layer="25" font="vector" ratio="20" rot="R90" align="bottom-center"/>
 <attribute name="VALUE" x="76.2" y="-100.33" size="0.6096" layer="27" font="vector" ratio="20" rot="R90" align="top-center"/>
 </element>
@@
 <contactref element="J9" pad="25"/>
 <contactref element="J8" pad="27"/>
+<wire x1="46.645" y1="3.66" x2="46.645" y2="9.365925" width="0.8128" layer="1"/>
+<wire x1="46.645" y1="9.365925" x2="45.7854625" y2="10.2254625" width="0.8128" layer="1"/>
 <wire x1="139.7" y1="48.0822" x2="143.505" y2="103.02" width="0" layer="19" extent="1-1"/>
-<wire x1="46.645" y1="3.66" x2="139.7" y2="48.0822" width="0" layer="19" extent="1-1"/>
+<wire x1="46.645" y1="9.365925" x2="139.7" y2="48.0822" width="0" layer="19" extent="1-1"/>
 <wire x1="81.432" y1="-124.46" x2="46.645" y2="3.66" width="0" layer="19" extent="1-1"/>
 </signal>
@@
 <contactref element="U6" pad="6"/>
 <contactref element="J8" pad="28"/>
-<wire x1="52.222" y1="-128.27" x2="142.24" y2="48.0822" width="0" layer="19" extent="1-1"/>
-<wire x1="49.415" y1="3.66" x2="52.222" y2="-128.27" width="0" layer="19" extent="1-1"/>
+<wire x1="49.415" y1="3.66" x2="49.415" y2="9.005" width="0.8128" layer="1"/>
+<wire x1="49.415" y1="9.005" x2="48.26" y2="10.16" width="0.8128" layer="1"/>
+<wire x1="49.415" y1="9.005" x2="142.24" y2="48.0822" width="0" layer="19" extent="1-1"/>
+<wire x1="52.222" y1="-128.27" x2="49.415" y2="3.66" width="0" layer="19" extent="1-1"/>
 </signal>
 <signal name="5V-DIG-TX-EN">
@@
 <contactref element="J8" pad="2"/>
 <contactref element="J9" pad="21"/>
+<wire x1="72.96" y1="6.5" x2="72.96" y2="9.46" width="0.8128" layer="1"/>
+<wire x1="72.96" y1="9.46" x2="73.66" y2="10.16" width="0.8128" layer="1"/>
 <wire x1="142.24" y1="53.5178" x2="132.425" y2="103.02" width="0" layer="19" extent="1-1"/>
-<wire x1="77.622" y1="-74.93" x2="142.24" y2="53.5178" width="0" layer="19" extent="1-1"/>
-<wire x1="72.96" y1="6.5" x2="77.622" y2="-74.93" width="0" layer="19" extent="1-1"/>
+<wire x1="73.66" y1="10.16" x2="142.24" y2="53.5178" width="0" layer="19" extent="1-1"/>
+<wire x1="77.622" y1="-74.93" x2="72.96" y2="6.5" width="0" layer="19" extent="1-1"/>
 </signal>
 <signal name="5V-ACT-LASER">
@@
 <contactref element="U6" pad="13"/>
 <contactref element="J8" pad="3"/>
-<wire x1="52.222" y1="-77.47" x2="139.7" y2="53.5178" width="0" layer="19" extent="1-1"/>
-<wire x1="70.19" y1="6.5" x2="52.222" y2="-77.47" width="0" layer="19" extent="1-1"/>
+<wire x1="70.19" y1="6.5" x2="70.19" y2="9.82" width="0.8128" layer="1"/>
+<wire x1="70.19" y1="9.82" x2="69.85" y2="10.16" width="0.8128" layer="1"/>
+<wire x1="70.19" y1="9.82" x2="139.7" y2="53.5178" width="0" layer="19" extent="1-1"/>
+<wire x1="52.222" y1="-77.47" x2="70.19" y2="6.5" width="0" layer="19" extent="1-1"/>
 </signal>
 <signal name="N$21">
@@
 <contactref element="J9" pad="24"/>
 <contactref element="J8" pad="23"/>
+<wire x1="35.565" y1="3.66" x2="35.565" y2="7.615" width="0.8128" layer="1"/>
+<wire x1="35.565" y1="7.615" x2="34.29" y2="8.89" width="0.8128" layer="1"/>
 <wire x1="139.7" y1="39.1922" x2="140.735" y2="103.02" width="0" layer="19" extent="1-1"/>
-<wire x1="81.432" y1="-99.06" x2="139.7" y2="39.1922" width="0" layer="19" extent="1-1"/>
-<wire x1="35.565" y1="3.66" x2="81.432" y2="-99.06" width="0" layer="19" extent="1-1"/>
+<wire x1="35.565" y1="7.615" x2="139.7" y2="39.1922" width="0" layer="19" extent="1-1"/>
+<wire x1="81.432" y1="-99.06" x2="35.565" y2="3.66" width="0" layer="19" extent="1-1"/>
 </signal>
 <signal name="5V-ACT-CAM">
@@
 <contactref element="U7" pad="6"/>
 <contactref element="J8" pad="24"/>
-<wire x1="49.682" y1="-95.25" x2="142.24" y2="39.1922" width="0" layer="19" extent="1-1"/>
-<wire x1="38.335" y1="3.66" x2="49.682" y2="-95.25" width="0" layer="19" extent="1-1"/>
+<wire x1="38.335" y1="3.66" x2="38.335" y2="8.655" width="0.8128" layer="1"/>
+<wire x1="38.335" y1="8.655" x2="36.83" y2="10.16" width="0.8128" layer="1"/>
+<wire x1="38.335" y1="8.655" x2="142.24" y2="39.1922" width="0" layer="19" extent="1-1"/>
+<wire x1="49.682" y1="-95.25" x2="38.335" y2="3.66" width="0" layer="19" extent="1-1"/>
 </signal>
 <signal name="5V-DIG-CAM-EN">
@@
 <contactref element="U9" pad="9"/>
 <contactref element="J8" pad="25"/>
+<wire x1="41.105" y1="3.66" x2="40.07561875" y2="3.66" width="0.8128" layer="1"/>
+<wire x1="40.07561875" y1="3.66" x2="38.84481875" y2="2.4292" width="0.8128" layer="1"/>
+<wire x1="38.84481875" y1="2.4292" x2="24.2408" y2="2.4292" width="0.8128" layer="1"/>
+<wire x1="24.2408" y1="2.4292" x2="21.59" y2="5.08" width="0.8128" layer="1"/>
 <wire x1="41.105" y1="3.66" x2="133.35" y2="44.6278" width="0" layer="19" extent="1-1"/>
-<wire x1="24.282" y1="-95.25" x2="41.105" y2="3.66" width="0" layer="19" extent="1-1"/>
+<wire x1="24.282" y1="-95.25" x2="24.2408" y2="2.4292" width="0" layer="19" extent="1-1"/>
 </signal>
 <signal name="12V-STA">
@@
 <contactref element="U9" pad="13"/>
 <contactref element="J8" pad="14"/>
-<wire x1="21.742" y1="-52.07" x2="130.81" y2="44.6278" width="0" layer="19" extent="1-1"/>
-<wire x1="39.72" y1="6.5" x2="21.742" y2="-52.07" width="0" layer="19" extent="1-1"/>
+<wire x1="39.72" y1="6.5" x2="38.3" y2="5.08" width="0.8128" layer="16"/>
+<wire x1="24.13" y1="5.08" x2="21.59" y2="7.62" width="0.8128" layer="16"/>
+<wire x1="38.3" y1="5.08" x2="24.13" y2="5.08" width="0.8128" layer="16"/>
+<wire x1="39.72" y1="6.5" x2="130.81" y2="44.6278" width="0" layer="19" extent="1-1"/>
+<wire x1="21.742" y1="-52.07" x2="24.13" y2="5.08" width="0" layer="19" extent="1-16"/>
 </signal>
 <signal name="5V-DIG-STA">
@@
 <contactref element="J9" pad="22"/>
 <contactref element="J8" pad="12"/>
+<wire x1="45.26" y1="6.5" x2="45.26" y2="9.35" width="0.8128" layer="1"/>
+<wire x1="45.26" y1="9.35" x2="44.45" y2="10.16" width="0.8128" layer="1"/>
 <wire x1="142.24" y1="44.6278" x2="135.195" y2="103.02" width="0" layer="19" extent="1-1"/>
-<wire x1="76.352" y1="-54.61" x2="142.24" y2="44.6278" width="0" layer="19" extent="1-1"/>
-<wire x1="45.26" y1="6.5" x2="76.352" y2="-54.61" width="0" layer="19" extent="1-1"/>
+<wire x1="45.26" y1="9.35" x2="142.24" y2="44.6278" width="0" layer="19" extent="1-1"/>
+<wire x1="76.352" y1="-54.61" x2="45.26" y2="6.5" width="0" layer="19" extent="1-1"/>
 </signal>
 <signal name="5V-ACT-STA">
@@
 <contactref element="U7" pad="13"/>
 <contactref element="J8" pad="13"/>
-<wire x1="57.302" y1="-53.34" x2="139.7" y2="44.6278" width="0" layer="19" extent="1-1"/>
-<wire x1="42.49" y1="6.5" x2="57.302" y2="-53.34" width="0" layer="19" extent="1-1"/>
+<wire x1="42.49" y1="6.5" x2="42.49" y2="9.58" width="0.8128" layer="1"/>
+<wire x1="42.49" y1="9.58" x2="41.91" y2="10.16" width="0.8128" layer="1"/>
+<wire x1="42.49" y1="9.58" x2="139.7" y2="44.6278" width="0" layer="19" extent="1-1"/>
+<wire x1="57.302" y1="-53.34" x2="42.49" y2="6.5" width="0" layer="19" extent="1-1"/>
 </signal>
 <signal name="5V-ACT-STA-EN">
@@
 <contactref element="U9" pad="6"/>
 <contactref element="J8" pad="19"/>
+<wire x1="25.87" y1="6.5" x2="24.75" y2="7.62" width="0.8128" layer="1"/>
+<wire x1="24.75" y1="7.62" x2="24.13" y2="7.62" width="0.8128" layer="1"/>
 <wire x1="47.142" y1="-30.48" x2="133.35" y2="39.1922" width="0" layer="19" extent="1-1"/>
-<wire x1="25.87" y1="6.5" x2="133.35" y2="39.1922" width="0" layer="19" extent="1-1"/>
+<wire x1="25.87" y1="6.5" x2="47.142" y2="-30.48" width="0" layer="19" extent="1-1"/>
 </signal>
 <signal name="5V-DIG-MAG">
@@
 <contactref element="J9" pad="23"/>
 <contactref element="J8" pad="18"/>
+<wire x1="28.64" y1="6.5" x2="28.64" y2="9.46" width="0.8128" layer="1"/>
+<wire x1="28.64" y1="9.46" x2="28.2456" y2="9.8544" width="0.8128" layer="1"/>
 <wire x1="130.81" y1="39.1922" x2="137.965" y2="103.02" width="0" layer="19" extent="1-1"/>
 <wire x1="80.162" y1="-27.94" x2="130.81" y2="39.1922" width="0" layer="19" extent="1-1"/>

Commit message: Replace resistor networks.
Parts:
- removed RN1: 100k, PowerManagementParts:SO16L
- removed RN2, RN3: 100Ω, PowerManagementParts:SO16L
- removed RN4: 100kΩ, PowerManagementParts:SO16L
- added R23, R25, R26, R27, R35, R36, R37, R38, R41, R42, R45, R46: 100k, rcl:R0805
- added R24, R28, R29, R30, R31, R32, R33, R34, R39, R40, R43, R44: 100Ω, rcl:R0805
Connections:
- net 12V: now also R45.2, R46.2; no longer RN4.13, RN4.14
- net 12V-CAM-EN: now also R43.1; no longer RN3.3
- net 12V-STA-EN: now also R44.1; no longer RN3.4
- net 5-ACT-LASER-EN: now also R30.1; no longer RN2.4
- net 5V-ACT: now also R25.2, R27.2, R36.2, R38.2, R42.2; no longer RN1.11, RN1.13, RN1.15, RN1.9, RN4.15
- net 5V-ACT-CAM-EN: now also R32.1; no longer RN2.6
- net 5V-ACT-MAG-EN: now also R40.1; no longer RN3.2
- net 5V-ACT-STA-EN: now also R34.1; no longer RN2.8
- net 5V-ACT-TX-EN: now also R28.1; no longer RN2.2
- net 5V-DIG: now also R23.2, R26.2, R35.2, R37.2, R41.2; no longer RN1.10, RN1.12, RN1.14, RN1.16, RN4.16
- net 5V-DIG-CAM-EN: now also R31.1; no longer RN2.5
- net 5V-DIG-LASER-EN: now also R29.1; no longer RN2.3
- net 5V-DIG-MAG-EN: now also R39.1; no longer RN3.1
- net 5V-DIG-STA-EN: now also R33.1; no longer RN2.7
- net 5V-DIG-TX-EN: now also R24.1; no longer RN2.1
- net N$10: now also R25.1, R28.2; no longer RN1.2, RN2.15
- net N$13: now also R26.1, R29.2; no longer RN1.3, RN2.14
- net N$15: now also R27.1, R30.2; no longer RN1.4, RN2.13
- net N$21: now also R40.2, R42.1; no longer RN3.15, RN4.2
- net N$23: now also R39.2, R41.1; no longer RN3.16, RN4.1
- net N$25: now also R34.2, R38.1; no longer RN1.8, RN2.9
- net N$27: now also R33.2, R37.1; no longer RN1.7, RN2.10
- net N$29: now also R32.2, R36.1; no longer RN1.6, RN2.11
- net N$31: now also R31.2, R35.1; no longer RN1.5, RN2.12
- net N$40: now also R43.2, R45.1; no longer RN3.14, RN4.3
- net N$43: now also R44.2, R46.1; no longer RN3.13, RN4.4
- net N$9: now also R23.1, R24.2; no longer RN1.1, RN2.16
Routing:
- net 12V-CAM: track 21.1 -> 0.00 mm
- net 12V-STA: track 19.8 -> 0.00 mm
- net GND: track 58.6 -> 47.4 mm
- net 5V-ACT-CAM: track 7.12 -> 0.00 mm
- net 5V-ACT-TX: track 6.98 -> 0.00 mm
- net 5V-DIG-TX: track 6.92 -> 0.00 mm
- net N$2: track 6.66 -> 0.00 mm
- net N$1: track 6.66 -> 0.00 mm
- net 5V-DIG-CAM: track 5.76 -> 0.00 mm
- net SUPPLY_FOR_5V-ACT: track 5.55 -> 0.00 mm
- net SUPPLY_FOR_12V: track 5.55 -> 0.00 mm
- net 5V-DIG-STA: track 4.00 -> 0.00 mm
- net 5V-DIG-LASER: track 3.95 -> 0.00 mm
- net 5V-ACT-STA: track 3.90 -> 0.00 mm
- net 5V-ACT-LASER: track 3.80 -> 0.00 mm
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
Commit message: Moved components around on board. Updated power input header
Parts:
- removed J7: (no value), SparkFun-Connectors:2X5
- added TP1: TPPAD1-13, testpad:P1-13
- moved R46 169.6 mm to (10.2, -48.0), turned to 180 degrees
- moved R42 144.0 mm to (31.8, -36.8), turned to 90 degrees
- moved R45 141.5 mm to (7.62, -100.3), turned to 90 degrees
- moved TP_5V-DIG_CTRL 123.3 mm to (-17.8, 61.0)
- moved C10 115.8 mm to (-17.8, 45.7)
- moved C8 115.8 mm to (-17.8, 55.9)
- moved C9 115.8 mm to (-17.8, 50.8)
- moved C2 99.2 mm to (-19.1, 86.4), turned to 90 degrees
- moved C7 97.9 mm to (-22.9, 86.4), turned to 90 degrees
- moved C1 78.8 mm to (-5.08, 31.8)
- moved TP_5V-ACT_CTRL 78.8 mm to (-21.6, 31.8)
- moved C6 36.4 mm to (34.3, 115.6)
- moved R5 30.5 mm to (108.0, 123.2)
- moved R6 30.5 mm to (113.0, 123.2)
- moved TP_12V_CTRL 30.5 mm to (-21.6, 36.8)
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Connections:
- removed net SUPPLY_FOR_12V: C3.1, J7.7, U4.1
- removed net SUPPLY_FOR_5V-ACT: C1.1, J7.5, U3.1
- new net SUPPLY_FOR_ACT: C1.1, C3.1, J1.10, U3.1, U4.1
- net 12V: no longer J7.10
- net 5V-ACT: no longer J7.8
- net 5V-DIG: no longer J7.6
- net GND: now also J1.12, J1.13, J1.14, J1.15, J1.5, J1.6, J1.7, J1.8, TP1.TP; no longer J7.1
- net MNGR-3.3V: no longer J7.4
- net MNGR-5V: no longer J7.2
- net SUPPLY_FOR_5V-DIG: now also J1.4; no longer J7.3
- net SUPPLY_FOR_MNGR: now also J1.1; no longer J7.9
Routing:
- net 12V: track 57.6 -> 4.98 mm
- net GND: track 47.4 -> 11.7 mm, vias 10 -> 3
- net 5V-ACT: track 37.4 -> 21.4 mm
- net N$4: track 12.9 -> 0.00 mm
- net SUPPLY_FOR_MNGR: track 8.90 -> 0.00 mm
- net N$3: track 8.01 -> 0.00 mm
- net MNGR-5V: track 26.0 -> 18.4 mm
- net N$5: track 6.79 -> 0.00 mm
- net N$36: track 6.20 -> 0.00 mm
- net N$20: track 4.13 -> 0.00 mm
- net N$19: track 4.13 -> 0.00 mm
- net N$18: track 4.13 -> 0.00 mm
- net N$17: track 4.13 -> 0.00 mm
