File: SafetySwitchBoard/SafetySwitchBoard.brd (EAGLE design)
At the start: 47 x 73.7 mm, 10 parts

Commit message: Refined SafetySwitchBoard
Parts:
- renumbered U$1 to 5V_CAM, U$2 to 5V_LASER, U$3 to 5V_TX, U$4 to 5V_STA, U$5 to 5V_MAG
Routing:
- added copper zone on layer 1, net GND
Other:
- board text added: "CSM Rocksat-x Rev1 01/30/2020 By: Graham Braly and Mark Gilliland"
Changed lines of the file:
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@@
 <wire x1="35.56" y1="6.35" x2="34.29" y2="7.62" width="1.016" layer="21"/>
 <wire x1="35.56" y1="6.35" x2="34.29" y2="5.08" width="1.016" layer="21"/>
+<text x="16.51" y="12.7" size="1.27" layer="21" rot="R90">CSM Rocksat-x
+Rev1 01/30/2020
+By: Graham Braly and Mark Gilliland</text>
 </plain>
 <attributes>
@@
 <attribute name="VALUE" x="57.62" y="1.08" size="1.778" layer="27" rot="R90"/>
 </element>
-<element name="U$1" library="PowerManagementParts" package="MTA106" value="MTA106" x="24.13" y="6.35" smashed="yes" rot="R270">
-<attribute name="NAME" x="30.988" y="10.668" size="1.27" layer="25" rot="R270"/>
-</element>
-<element name="U$2" library="PowerManagementParts" package="MTA106" value="MTA106" x="24.13" y="16.51" smashed="yes" rot="R270">
-<attribute name="NAME" x="30.988" y="19.685" size="1.27" layer="25" rot="R270"/>
-</element>
-<element name="U$3" library="PowerManagementParts" package="MTA106" value="MTA106" x="24.13" y="26.67" smashed="yes" rot="R270">
-<attribute name="NAME" x="30.988" y="29.845" size="1.27" layer="25" rot="R270"/>
-</element>
-<element name="U$4" library="PowerManagementParts" package="MTA106" value="MTA106" x="24.13" y="36.83" smashed="yes" rot="R270">
+<element name="5V_CAM" library="PowerManagementParts" package="MTA106" value="MTA106" x="24.13" y="6.35" smashed="yes" rot="R270">
+<attribute name="NAME" x="30.988" y="9.906" size="1.27" layer="25" rot="R270"/>
+</element>
+<element name="5V_LASER" library="PowerManagementParts" package="MTA106" value="MTA106" x="24.13" y="16.51" smashed="yes" rot="R270">
+<attribute name="NAME" x="30.988" y="20.955" size="1.27" layer="25" rot="R270"/>
+</element>
+<element name="5V_TX" library="PowerManagementParts" package="MTA106" value="MTA106" x="24.13" y="26.67" smashed="yes" rot="R270">
+<attribute name="NAME" x="30.988" y="29.464" size="1.27" layer="25" rot="R270"/>
+</element>
+<element name="5V_STA" library="PowerManagementParts" package="MTA106" value="MTA106" x="24.13" y="36.83" smashed="yes" rot="R270">
 <attribute name="NAME" x="30.988" y="40.005" size="1.27" layer="25" rot="R270"/>
 </element>
-<element name="U$5" library="PowerManagementParts" package="MTA106" value="MTA106" x="24.13" y="46.99" smashed="yes" rot="R270">
-<attribute name="NAME" x="30.988" y="50.165" size="1.27" layer="25" rot="R270"/>
+<element name="5V_MAG" library="PowerManagementParts" package="MTA106" value="MTA106" x="24.13" y="46.99" smashed="yes" rot="R270">
+<attribute name="NAME" x="31.115" y="50.546" size="1.27" layer="25" rot="R270"/>
 </element>
 <element name="12V_CAM" library="PowerManagementParts" package="MTA106" value="MTA106" x="24.13" y="57.15" smashed="yes" rot="R270">
@@
 <contactref element="INPUT-DSUB" pad="25"/>
 <contactref element="OUTPUT-DSUB" pad="32"/>
+<polygon width="0.1524" layer="1">
+<vertex x="0" y="0"/>
+<vertex x="46.99" y="0"/>
+<vertex x="46.99" y="73.66"/>
+<vertex x="0" y="73.66"/>
+</polygon>
 </signal>
 <signal name="LASER-UART-1">
@@
 <signal name="5V-ACT-CAM">
 <contactref element="INPUT-DSUB" pad="13"/>
-<contactref element="U$1" pad="P$1"/>
+<contactref element="5V_CAM" pad="P$1"/>
 <wire x1="9.04" y1="45.14" x2="9.6463" y2="44.5337" width="2.286" layer="1"/>
 <wire x1="9.6463" y1="44.5337" x2="9.9362375" y2="44.5337" width="2.286" layer="1"/>
@@
 <signal name="5V-ACT-LASER">
 <contactref element="INPUT-DSUB" pad="14"/>
-<contactref element="U$2" pad="P$1"/>
+<contactref element="5V_LASER" pad="P$1"/>
 <wire x1="9.04" y1="47.91" x2="9.27" y2="47.68" width="2.286" layer="1"/>
 <wire x1="9.27" y1="47.68" x2="10.38204375" y2="47.68" width="2.286" layer="1"/>
@@
 <signal name="5V-ACT-TX">
 <contactref element="INPUT-DSUB" pad="15"/>
-<contactref element="U$3" pad="P$1"/>
+<contactref element="5V_TX" pad="P$1"/>
 <wire x1="9.04" y1="50.68" x2="9.27" y2="50.45" width="2.286" layer="1"/>
 <wire x1="9.27" y1="50.45" x2="11.20415" y2="50.45" width="2.286" layer="1"/>
@@
 <signal name="5V-ACT-STA">
 <contactref element="INPUT-DSUB" pad="16"/>
-<contactref element="U$4" pad="P$1"/>
+<contactref element="5V_STA" pad="P$1"/>
 <via x="24.13" y="41.91" extent="1-16" drill="0.85"/>
 <wire x1="9.04" y1="53.45" x2="9.6463" y2="52.8437" width="2.286" layer="16"/>
@@
 <signal name="5V-ACT-MAG">
 <contactref element="INPUT-DSUB" pad="17"/>
-<contactref element="U$5" pad="P$1"/>
+<contactref element="5V_MAG" pad="P$1"/>
 <wire x1="16.53864375" y1="56.22" x2="18.85984375" y2="53.8988" width="2.286" layer="1"/>
 <wire x1="18.85984375" y1="53.8988" x2="21.0312" y2="53.8988" width="2.286" layer="1"/>
@@
 </signal>
 <signal name="5V-ACT-CAM-SWITCHED">
-<contactref element="U$1" pad="P$2"/>
+<contactref element="5V_CAM" pad="P$2"/>
 <contactref element="OUTPUT-DSUB" pad="7"/>
 <wire x1="33.528" y1="29.718" x2="35.56" y2="31.75" width="2.286" layer="1"/>
@@
 </signal>
 <signal name="5V-ACT-LASER-SWITCHED">
-<contactref element="U$2" pad="P$2"/>
+<contactref element="5V_LASER" pad="P$2"/>
 <contactref element="OUTPUT-DSUB" pad="6"/>
 <wire x1="28.448" y1="16.51" x2="30.988" y2="19.05" width="2.286" layer="1"/>
@@
 </signal>
 <signal name="5V-ACT-TX-SWITCHED">
-<contactref element="U$3" pad="P$2"/>
+<contactref element="5V_TX" pad="P$2"/>
 <contactref element="OUTPUT-DSUB" pad="5"/>
 <wire x1="28.448" y1="32.258" x2="28.448" y2="26.67" width="2.286" layer="1"/>
@@
 </signal>
 <signal name="5V-ACT-MAG-SWITCHED">
-<contactref element="U$5" pad="P$2"/>
+<contactref element="5V_MAG" pad="P$2"/>
 <contactref element="OUTPUT-DSUB" pad="3"/>
 <wire x1="28.448" y1="46.99" x2="28.448" y2="51.308" width="2.286" layer="16"/>
@@
 </signal>
 <signal name="5V-ACT-STA-SWITCHED">
-<contactref element="U$4" pad="P$2"/>
+<contactref element="5V_STA" pad="P$2"/>
 <contactref element="OUTPUT-DSUB" pad="4"/>
 <wire x1="28.448" y1="36.83" x2="28.448" y2="43.18" width="2.286" layer="1"/>
@@
 </drawing>
 <compatibility>
+<note version="6.3" minversion="6.2.2" severity="warning">
+Since Version 6.2.2 text objects can contain more than one line,
+which will not be processed correctly with this version.
+</note>
 <note version="8.2" severity="warning">
 Since Version 8.2, EAGLE supports online libraries. The ids
