File: SafetySwitchBoard/SafetySwitchBoard.sch (EAGLE design)
At the start: 10 parts

Commit message: Refined SafetySwitchBoard
Parts:
- renumbered U$1 to 5V_CAM, U$2 to 5V_LASER, U$3 to 5V_TX, U$4 to 5V_STA, U$5 to 5V_MAG
Changed lines of the file:
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@@
 <part name="FRAME1" library="SparkFun-Aesthetics" deviceset="FRAME-LETTER" device="NO_PACKAGE"/>
 <part name="OUTPUT-DSUB" library="D-Sub Connectors" library_urn="urn:adsk.eagle:library:11816059" deviceset="182-037-213R531" device="" package3d_urn="urn:adsk.eagle:package:11705754/3"/>
-<part name="U$1" library="PowerManagementParts" deviceset="MTA106" device=""/>
-<part name="U$2" library="PowerManagementParts" deviceset="MTA106" device=""/>
-<part name="U$3" library="PowerManagementParts" deviceset="MTA106" device=""/>
-<part name="U$4" library="PowerManagementParts" deviceset="MTA106" device=""/>
-<part name="U$5" library="PowerManagementParts" deviceset="MTA106" device=""/>
+<part name="5V_CAM" library="PowerManagementParts" deviceset="MTA106" device=""/>
+<part name="5V_LASER" library="PowerManagementParts" deviceset="MTA106" device=""/>
+<part name="5V_TX" library="PowerManagementParts" deviceset="MTA106" device=""/>
+<part name="5V_STA" library="PowerManagementParts" deviceset="MTA106" device=""/>
+<part name="5V_MAG" library="PowerManagementParts" deviceset="MTA106" device=""/>
 <part name="12V_CAM" library="PowerManagementParts" deviceset="MTA106" device=""/>
 <part name="12V_STA" library="PowerManagementParts" deviceset="MTA106" device=""/>
@@
 <attribute name="VALUE" x="125.984" y="25.4" size="1.778" layer="96" rot="MR0"/>
 </instance>
-<instance part="U$1" gate="G$1" x="215.9" y="175.26" smashed="yes">
+<instance part="5V_CAM" gate="G$1" x="215.9" y="175.26" smashed="yes">
 <attribute name="NAME" x="217.17" y="178.308" size="1.778" layer="95" font="vector" align="bottom-center"/>
 <attribute name="VALUE" x="216.916" y="171.958" size="1.778" layer="96" font="vector" align="top-center"/>
 </instance>
-<instance part="U$2" gate="G$1" x="215.9" y="160.02" smashed="yes">
+<instance part="5V_LASER" gate="G$1" x="215.9" y="160.02" smashed="yes">
 <attribute name="NAME" x="217.17" y="163.068" size="1.778" layer="95" font="vector" align="bottom-center"/>
 <attribute name="VALUE" x="216.916" y="156.718" size="1.778" layer="96" font="vector" align="top-center"/>
 </instance>
-<instance part="U$3" gate="G$1" x="215.9" y="144.78" smashed="yes">
+<instance part="5V_TX" gate="G$1" x="215.9" y="144.78" smashed="yes">
 <attribute name="NAME" x="217.17" y="147.828" size="1.778" layer="95" font="vector" align="bottom-center"/>
 <attribute name="VALUE" x="216.916" y="141.478" size="1.778" layer="96" font="vector" align="top-center"/>
 </instance>
-<instance part="U$4" gate="G$1" x="215.9" y="129.54" smashed="yes">
+<instance part="5V_STA" gate="G$1" x="215.9" y="129.54" smashed="yes">
 <attribute name="NAME" x="217.17" y="132.588" size="1.778" layer="95" font="vector" align="bottom-center"/>
 <attribute name="VALUE" x="216.916" y="126.238" size="1.778" layer="96" font="vector" align="top-center"/>
 </instance>
-<instance part="U$5" gate="G$1" x="215.9" y="114.3" smashed="yes">
+<instance part="5V_MAG" gate="G$1" x="215.9" y="114.3" smashed="yes">
 <attribute name="NAME" x="217.17" y="117.348" size="1.778" layer="95" font="vector" align="bottom-center"/>
 <attribute name="VALUE" x="216.916" y="110.998" size="1.778" layer="96" font="vector" align="top-center"/>
@@
 </segment>
 <segment>
-<pinref part="U$1" gate="G$1" pin="P"/>
+<pinref part="5V_CAM" gate="G$1" pin="P"/>
 <wire x1="213.36" y1="175.26" x2="210.82" y2="175.26" width="0.1524" layer="91"/>
 <label x="210.82" y="175.26" size="1.27" layer="95" rot="R180" xref="yes"/>
@@
 </segment>
 <segment>
-<pinref part="U$2" gate="G$1" pin="P"/>
+<pinref part="5V_LASER" gate="G$1" pin="P"/>
 <wire x1="213.36" y1="160.02" x2="210.82" y2="160.02" width="0.1524" layer="91"/>
 <label x="210.82" y="160.02" size="1.27" layer="95" rot="R180" xref="yes"/>
@@
 </segment>
 <segment>
-<pinref part="U$3" gate="G$1" pin="P"/>
+<pinref part="5V_TX" gate="G$1" pin="P"/>
 <wire x1="213.36" y1="144.78" x2="210.82" y2="144.78" width="0.1524" layer="91"/>
 <label x="210.82" y="144.78" size="1.27" layer="95" rot="R180" xref="yes"/>
@@
 </segment>
 <segment>
-<pinref part="U$4" gate="G$1" pin="P"/>
+<pinref part="5V_STA" gate="G$1" pin="P"/>
 <wire x1="213.36" y1="129.54" x2="210.82" y2="129.54" width="0.1524" layer="91"/>
 <label x="210.82" y="129.54" size="1.27" layer="95" rot="R180" xref="yes"/>
@@
 </segment>
 <segment>
-<pinref part="U$5" gate="G$1" pin="P"/>
+<pinref part="5V_MAG" gate="G$1" pin="P"/>
 <wire x1="213.36" y1="114.3" x2="210.82" y2="114.3" width="0.1524" layer="91"/>
 <label x="210.82" y="114.3" size="1.27" layer="95" rot="R180" xref="yes"/>
@@
 <net name="5V-ACT-CAM-SWITCHED" class="0">
 <segment>
-<pinref part="U$1" gate="G$1" pin="O"/>
+<pinref part="5V_CAM" gate="G$1" pin="O"/>
 <wire x1="220.98" y1="177.8" x2="223.52" y2="177.8" width="0.1524" layer="91"/>
 <label x="223.52" y="177.8" size="1.27" layer="95" xref="yes"/>
@@
 <net name="5V-ACT-LASER-SWITCHED" class="0">
 <segment>
-<pinref part="U$2" gate="G$1" pin="O"/>
+<pinref part="5V_LASER" gate="G$1" pin="O"/>
 <wire x1="220.98" y1="162.56" x2="223.52" y2="162.56" width="0.1524" layer="91"/>
 <label x="223.52" y="162.56" size="1.27" layer="95" xref="yes"/>
@@
 <net name="5V-ACT-TX-SWITCHED" class="0">
 <segment>
-<pinref part="U$3" gate="G$1" pin="O"/>
+<pinref part="5V_TX" gate="G$1" pin="O"/>
 <wire x1="220.98" y1="147.32" x2="223.52" y2="147.32" width="0.1524" layer="91"/>
 <label x="223.52" y="147.32" size="1.27" layer="95" xref="yes"/>
@@
 <net name="5V-ACT-MAG-SWITCHED" class="0">
 <segment>
-<pinref part="U$5" gate="G$1" pin="O"/>
+<pinref part="5V_MAG" gate="G$1" pin="O"/>
 <wire x1="220.98" y1="116.84" x2="223.52" y2="116.84" width="0.1524" layer="91"/>
 <label x="223.52" y="116.84" size="1.27" layer="95" xref="yes"/>
@@
 <net name="5V-ACT-STA-SWITCHED" class="0">
 <segment>
-<pinref part="U$4" gate="G$1" pin="O"/>
+<pinref part="5V_STA" gate="G$1" pin="O"/>
 <wire x1="220.98" y1="132.08" x2="223.52" y2="132.08" width="0.1524" layer="91"/>
 <label x="223.52" y="132.08" size="1.27" layer="95" xref="yes"/>
