File: DataControlBoard/DataControlBoard-RPi/DataControlBoard-RPi.brd (EAGLE design)
At the start: 66 x 30.5 mm, 21 parts, among them J1 USB3150-30-130-AMANUFACTURABLE, J1-L-DATA USB3150-30-130-AMANUFACTURABLE, J2 USB3150-30-130-AMANUFACTURABLE, J2-L-PWR USB3150-30-130-AMANUFACTURABLE, J3-M-DATA USB3150-30-130-AMANUFACTURABLE, J4-M-PWR USB3150-30-130-AMANUFACTURABLE, J5-S-DATA USB3150-30-130-AMANUFACTURABLE, J6-S-PWR USB3150-30-130-AMANUFACTURABLE, J7 FEMALE 2x3, J8 USB3150-30-130-AMANUFACTURABLE

Commit message: Finished RPi board rev 2.
Connections:
- net GND: now also J1-L-DATA.P$1, J1.P$1, J2-L-PWR.P$1, J2.P$1, J3-M-DATA.P$1, J4-M-PWR.P$1, J5-S-DATA.P$1, J6-S-PWR.P$1, J8.P$1; no longer J1-L-DATA.S1, J1-L-DATA.S2, J1.S1, J1.S2, J2-L-PWR.S1, J2-L-PWR.S2, J2.S1, J2.S2, J3-M-DATA.S1, J3-M-DATA.S2, J4-M-PWR.S1, J4-M-PWR.S2, J5-S-DATA.S1, J5-S-DATA.S2, J6-S-PWR.S1, J6-S-PWR.S2, J8.S1, J8.S2
Routing:
- added copper zone on layer 1, net GND
Other:
- outline, holes or cut-outs redrawn
- board text added: "Rev 2.0"
- board text removed: "Rev 1.0"
Changed lines of the file:
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@@
 <setting verticaltext="up"/>
 </settings>
-<grid distance="10" unitdist="mil" unit="mil" style="lines" multiple="1" display="yes" altdistance="2.5" altunitdist="mil" altunit="mil"/>
+<grid distance="25" unitdist="mil" unit="mil" style="lines" multiple="1" display="yes" altdistance="2.5" altunitdist="mil" altunit="mil"/>
 <layers>
 <layer number="1" name="Top" color="4" fill="1" visible="yes" active="yes"/>
@@
 <layer number="115" name="ReferenceISLANDS" color="7" fill="1" visible="no" active="yes"/>
 <layer number="116" name="Patch_BOT" color="9" fill="4" visible="no" active="yes"/>
+<layer number="117" name="BACKMAAT1" color="7" fill="1" visible="no" active="no"/>
 <layer number="118" name="Rect_Pads" color="7" fill="1" visible="no" active="yes"/>
+<layer number="119" name="KAP_TEKEN" color="7" fill="1" visible="no" active="no"/>
+<layer number="120" name="KAP_MAAT1" color="7" fill="1" visible="no" active="no"/>
 <layer number="121" name="_tsilk" color="7" fill="1" visible="no" active="yes"/>
 <layer number="122" name="_bsilk" color="7" fill="1" visible="no" active="yes"/>
@@
 <layer number="128" name="_bValues" color="7" fill="1" visible="no" active="yes"/>
 <layer number="129" name="Mask" color="7" fill="1" visible="no" active="yes"/>
+<layer number="130" name="SMDSTROOK" color="7" fill="1" visible="no" active="no"/>
 <layer number="131" name="tAdjust" color="7" fill="1" visible="no" active="yes"/>
 <layer number="132" name="bAdjust" color="7" fill="1" visible="no" active="yes"/>
+<layer number="133" name="bottom_silk" color="7" fill="1" visible="no" active="no"/>
 <layer number="144" name="Drill_legend" color="7" fill="1" visible="no" active="yes"/>
 <layer number="150" name="Notes" color="7" fill="1" visible="no" active="yes"/>
@@
 Mark Gilliland, Graham Braly
 2019 Mines RockSat-X</text>
-<text x="22.733" y="11.303" size="1.778" layer="25">Rev 1.0</text>
+<text x="24.003" y="11.938" size="1.778" layer="25">Rev 2.0</text>
 <text x="33.782" y="20.828" size="1.016" layer="25" font="vector" rot="R270">Boom
 Cam
@@
 <text x="34.798" y="11.43" size="1.016" layer="25" font="vector" rot="R270">Magnet
 USB</text>
-<text x="1.778" y="9.398" size="1.778" layer="51">1   2   3</text>
+<text x="1.778" y="9.398" size="1.27" layer="51">1   2   3</text>
+<wire x1="8.255" y1="29.21" x2="8.255" y2="10.16" width="0.1524" layer="20"/>
+<wire x1="8.255" y1="10.16" x2="22.86" y2="10.16" width="0.1524" layer="20"/>
+<wire x1="22.86" y1="10.16" x2="22.86" y2="29.21" width="0.1524" layer="20"/>
+<wire x1="22.86" y1="29.21" x2="8.255" y2="29.21" width="0.1524" layer="20"/>
 </plain>
 <attributes>
@@
 <contactref element="J8" pad="S3"/>
 <contactref element="J8" pad="S6"/>
-<contactref element="J8" pad="S2"/>
 <contactref element="J8" pad="S4"/>
 <contactref element="J8" pad="S5"/>
-<contactref element="J8" pad="S1"/>
-<polygon width="0.1524" layer="16">
+<polygon width="0.1524" layer="16" isolate="0.3048">
 <vertex x="66.04" y="0"/>
 <vertex x="0" y="0"/>
@@
 <contactref element="J5-S-DATA" pad="S3"/>
 <contactref element="J5-S-DATA" pad="S6"/>
-<contactref element="J5-S-DATA" pad="S2"/>
 <contactref element="J5-S-DATA" pad="S4"/>
 <contactref element="J5-S-DATA" pad="S5"/>
-<contactref element="J5-S-DATA" pad="S1"/>
 <contactref element="J3-M-DATA" pad="5"/>
 <contactref element="J3-M-DATA" pad="S3"/>
 <contactref element="J3-M-DATA" pad="S6"/>
-<contactref element="J3-M-DATA" pad="S2"/>
 <contactref element="J3-M-DATA" pad="S4"/>
 <contactref element="J3-M-DATA" pad="S5"/>
-<contactref element="J3-M-DATA" pad="S1"/>
 <contactref element="J1-L-DATA" pad="5"/>
 <contactref element="J1-L-DATA" pad="S3"/>
 <contactref element="J1-L-DATA" pad="S6"/>
-<contactref element="J1-L-DATA" pad="S2"/>
 <contactref element="J1-L-DATA" pad="S4"/>
 <contactref element="J1-L-DATA" pad="S5"/>
-<contactref element="J1-L-DATA" pad="S1"/>
 <contactref element="J2-L-PWR" pad="S3"/>
 <contactref element="J2-L-PWR" pad="S6"/>
-<contactref element="J2-L-PWR" pad="S2"/>
 <contactref element="J2-L-PWR" pad="S4"/>
 <contactref element="J2-L-PWR" pad="S5"/>
-<contactref element="J2-L-PWR" pad="S1"/>
 <contactref element="J2-L-PWR" pad="5"/>
 <contactref element="J4-M-PWR" pad="5"/>
 <contactref element="J4-M-PWR" pad="S3"/>
 <contactref element="J4-M-PWR" pad="S6"/>
-<contactref element="J4-M-PWR" pad="S2"/>
 <contactref element="J4-M-PWR" pad="S4"/>
 <contactref element="J4-M-PWR" pad="S5"/>
-<contactref element="J4-M-PWR" pad="S1"/>
 <contactref element="J6-S-PWR" pad="S3"/>
 <contactref element="J6-S-PWR" pad="S6"/>
-<contactref element="J6-S-PWR" pad="S2"/>
 <contactref element="J6-S-PWR" pad="S4"/>
 <contactref element="J6-S-PWR" pad="S5"/>
-<contactref element="J6-S-PWR" pad="S1"/>
 <contactref element="J6-S-PWR" pad="5"/>
 <contactref element="J1" pad="5"/>
-<contactref element="J1" pad="S1"/>
-<contactref element="J1" pad="S2"/>
 <contactref element="J1" pad="S3"/>
 <contactref element="J1" pad="S4"/>
@@
 <contactref element="J1" pad="S6"/>
 <contactref element="J2" pad="5"/>
-<contactref element="J2" pad="S1"/>
-<contactref element="J2" pad="S2"/>
 <contactref element="J2" pad="S3"/>
 <contactref element="J2" pad="S4"/>
@@
 <contactref element="J3" pad="3"/>
 <contactref element="J3" pad="5"/>
+<polygon width="0.1524" layer="1" isolate="0.3048">
+<vertex x="0" y="30.48"/>
+<vertex x="0" y="0"/>
+<vertex x="66.04" y="0"/>
+<vertex x="66.04" y="30.48"/>
+</polygon>
+<contactref element="J1-L-DATA" pad="P$1"/>
+<contactref element="J2-L-PWR" pad="P$1"/>
+<contactref element="J3-M-DATA" pad="P$1"/>
+<contactref element="J4-M-PWR" pad="P$1"/>
+<contactref element="J5-S-DATA" pad="P$1"/>
+<contactref element="J6-S-PWR" pad="P$1"/>
+<contactref element="J8" pad="P$1"/>
+<contactref element="J1" pad="P$1"/>
+<contactref element="J2" pad="P$1"/>
 </signal>
 <signal name="5V-DIG-MAG">
