File: DataControlBoard/DataControlBoard-RPi/DataControlBoard-RPi.sch (EAGLE design)
At the start: 18 parts, among them J1 USB3150-30-130-AMANUFACTURABLE, J1-L-DATA USB3150-30-130-AMANUFACTURABLE, J2 USB3150-30-130-AMANUFACTURABLE, J2-L-PWR USB3150-30-130-AMANUFACTURABLE, J3-M-DATA USB3150-30-130-AMANUFACTURABLE, J4-M-PWR USB3150-30-130-AMANUFACTURABLE, J5-S-DATA USB3150-30-130-AMANUFACTURABLE, J6-S-PWR USB3150-30-130-AMANUFACTURABLE, J7 FEMALE 2x3, J8 USB3150-30-130-AMANUFACTURABLE

Commit message: Ready for Diff Pair routing
Connections:
- net LIDAR-D+ renamed LIDAR-D_P
- net LIDAR-D- renamed LIDAR-D_N
- net MAG-D+ renamed MAG-D_P
- net MAG-D- renamed MAG-D_N
- net STA-D+ renamed STA-D_P
- net STA-D- renamed STA-D_N
Changed lines of the file:
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@@
 <class number="0" name="default" width="0" drill="0">
+</class>
+<class number="1" name="USB_diff" width="0.8128" drill="0">
+<clearance class="1" value="0.2032"/>
 </class>
 </classes>
@@
 </segment>
 </net>
-<net name="LIDAR-D-" class="0">
+<net name="LIDAR-D_P" class="0">
+<segment>
+<pinref part="J8" gate="G$1" pin="D+"/>
+<wire x1="30.48" y1="149.86" x2="25.4" y2="149.86" width="0.1524" layer="91"/>
+<label x="25.4" y="149.86" size="1.778" layer="95" rot="R180"/>
+</segment>
+<segment>
+<pinref part="J1-L-DATA" gate="G$1" pin="D+"/>
+<wire x1="154.94" y1="152.4" x2="152.4" y2="152.4" width="0.1524" layer="91"/>
+<label x="152.4" y="152.4" size="1.778" layer="95" rot="R180"/>
+</segment>
+</net>
+<net name="MAG-D_P" class="0">
+<segment>
+<pinref part="J1" gate="G$1" pin="D+"/>
+<wire x1="76.2" y1="149.86" x2="73.66" y2="149.86" width="0.1524" layer="91"/>
+<label x="73.66" y="149.86" size="1.778" layer="95" rot="R180"/>
+</segment>
+<segment>
+<pinref part="J3-M-DATA" gate="G$1" pin="D+"/>
+<wire x1="154.94" y1="114.3" x2="152.4" y2="114.3" width="0.1524" layer="91"/>
+<label x="152.4" y="114.3" size="1.778" layer="95" rot="R180"/>
+</segment>
+</net>
+<net name="USB-5V-MAG" class="0">
+<segment>
+<pinref part="J1" gate="G$1" pin="VBUS"/>
+<wire x1="76.2" y1="154.94" x2="73.66" y2="154.94" width="0.1524" layer="91"/>
+<label x="73.66" y="154.94" size="1.778" layer="95" rot="R180"/>
+</segment>
+<segment>
+<pinref part="J3-M-DATA" gate="G$1" pin="VBUS"/>
+<wire x1="154.94" y1="119.38" x2="152.4" y2="119.38" width="0.1524" layer="91"/>
+<label x="152.4" y="119.38" size="1.778" layer="95" rot="R180"/>
+</segment>
+</net>
+<net name="STA-D_N" class="0">
+<segment>
+<pinref part="J2" gate="G$1" pin="D-"/>
+<wire x1="76.2" y1="127" x2="73.66" y2="127" width="0.1524" layer="91"/>
+<label x="73.66" y="127" size="1.778" layer="95" rot="R180"/>
+</segment>
+<segment>
+<pinref part="J5-S-DATA" gate="G$1" pin="D-"/>
+<wire x1="154.94" y1="81.28" x2="152.4" y2="81.28" width="0.1524" layer="91"/>
+<label x="152.4" y="81.28" size="1.778" layer="95" rot="R180"/>
+</segment>
+</net>
+<net name="USB-5V-STA" class="0">
+<segment>
+<pinref part="J2" gate="G$1" pin="VBUS"/>
+<wire x1="76.2" y1="129.54" x2="73.66" y2="129.54" width="0.1524" layer="91"/>
+<label x="73.66" y="129.54" size="1.778" layer="95" rot="R180"/>
+</segment>
+<segment>
+<pinref part="J5-S-DATA" gate="G$1" pin="VBUS"/>
+<wire x1="154.94" y1="83.82" x2="152.4" y2="83.82" width="0.1524" layer="91"/>
+<label x="152.4" y="83.82" size="1.778" layer="95" rot="R180"/>
+</segment>
+</net>
+<net name="USB-5V-LID" class="0">
+<segment>
+<pinref part="J8" gate="G$1" pin="VBUS"/>
+<wire x1="30.48" y1="154.94" x2="25.4" y2="154.94" width="0.1524" layer="91"/>
+<label x="25.4" y="154.94" size="1.778" layer="95" rot="R180"/>
+</segment>
+<segment>
+<pinref part="J1-L-DATA" gate="G$1" pin="VBUS"/>
+<wire x1="154.94" y1="157.48" x2="152.4" y2="157.48" width="0.1524" layer="91"/>
+<label x="152.4" y="157.48" size="1.778" layer="95" rot="R180"/>
+</segment>
+</net>
+<net name="N$2" class="0">
+<segment>
+<pinref part="J3" gate="G$1" pin="2"/>
+<pinref part="TP1" gate="G$1" pin="TP"/>
+<wire x1="60.96" y1="50.8" x2="68.58" y2="50.8" width="0.1524" layer="91"/>
+</segment>
+</net>
+<net name="N$3" class="0">
+<segment>
+<pinref part="J3" gate="G$1" pin="4"/>
+<pinref part="TP2" gate="G$1" pin="TP"/>
+<wire x1="60.96" y1="48.26" x2="71.12" y2="48.26" width="0.1524" layer="91"/>
+</segment>
+</net>
+<net name="N$4" class="0">
+<segment>
+<pinref part="J3" gate="G$1" pin="6"/>
+<pinref part="TP3" gate="G$1" pin="TP"/>
+<wire x1="60.96" y1="45.72" x2="73.66" y2="45.72" width="0.1524" layer="91"/>
+</segment>
+</net>
+<net name="MAG-D_N" class="0">
+<segment>
+<pinref part="J3-M-DATA" gate="G$1" pin="D-"/>
+<wire x1="154.94" y1="116.84" x2="152.4" y2="116.84" width="0.1524" layer="91"/>
+<label x="152.4" y="116.84" size="1.778" layer="95" rot="R180"/>
+</segment>
+<segment>
+<pinref part="J1" gate="G$1" pin="D-"/>
+<wire x1="76.2" y1="152.4" x2="73.66" y2="152.4" width="0.1524" layer="91"/>
+<label x="73.66" y="152.4" size="1.778" layer="95" rot="R180"/>
+</segment>
+</net>
+<net name="STA-D_P" class="0">
+<segment>
+<pinref part="J2" gate="G$1" pin="D+"/>
+<wire x1="76.2" y1="124.46" x2="73.66" y2="124.46" width="0.1524" layer="91"/>
+<label x="73.66" y="124.46" size="1.778" layer="95" rot="R180"/>
+</segment>
+<segment>
+<pinref part="J5-S-DATA" gate="G$1" pin="D+"/>
+<wire x1="154.94" y1="78.74" x2="152.4" y2="78.74" width="0.1524" layer="91"/>
+<label x="152.4" y="78.74" size="1.778" layer="95" rot="R180"/>
+</segment>
+</net>
+<net name="LIDAR-D_N" class="0">
+<segment>
+<pinref part="J1-L-DATA" gate="G$1" pin="D-"/>
+<wire x1="154.94" y1="154.94" x2="152.4" y2="154.94" width="0.1524" layer="91"/>
+<label x="152.4" y="154.94" size="1.778" layer="95" rot="R180"/>
+</segment>
 <segment>
 <pinref part="J8" gate="G$1" pin="D-"/>
@@
 <label x="25.4" y="152.4" size="1.778" layer="95" rot="R180"/>
 </segment>
-<segment>
-<pinref part="J1-L-DATA" gate="G$1" pin="D-"/>
-<wire x1="154.94" y1="154.94" x2="152.4" y2="154.94" width="0.1524" layer="91"/>
-<label x="152.4" y="154.94" size="1.778" layer="95" rot="R180"/>
-</segment>
-</net>
-<net name="LIDAR-D+" class="0">
-<segment>
-<pinref part="J8" gate="G$1" pin="D+"/>
-<wire x1="30.48" y1="149.86" x2="25.4" y2="149.86" width="0.1524" layer="91"/>
-<label x="25.4" y="149.86" size="1.778" layer="95" rot="R180"/>
-</segment>
-<segment>
-<pinref part="J1-L-DATA" gate="G$1" pin="D+"/>
-<wire x1="154.94" y1="152.4" x2="152.4" y2="152.4" width="0.1524" layer="91"/>
-<label x="152.4" y="152.4" size="1.778" layer="95" rot="R180"/>
-</segment>
-</net>
-<net name="MAG-D+" class="0">
-<segment>
-<pinref part="J1" gate="G$1" pin="D+"/>
-<wire x1="76.2" y1="149.86" x2="73.66" y2="149.86" width="0.1524" layer="91"/>
-<label x="73.66" y="149.86" size="1.778" layer="95" rot="R180"/>
-</segment>
-<segment>
-<pinref part="J3-M-DATA" gate="G$1" pin="D+"/>
-<wire x1="154.94" y1="114.3" x2="152.4" y2="114.3" width="0.1524" layer="91"/>
-<label x="152.4" y="114.3" size="1.778" layer="95" rot="R180"/>
-</segment>
-</net>
-<net name="MAG-D-" class="0">
-<segment>
-<pinref part="J1" gate="G$1" pin="D-"/>
-<wire x1="76.2" y1="152.4" x2="73.66" y2="152.4" width="0.1524" layer="91"/>
-<label x="73.66" y="152.4" size="1.778" layer="95" rot="R180"/>
-</segment>
-<segment>
-<pinref part="J3-M-DATA" gate="G$1" pin="D-"/>
-<wire x1="154.94" y1="116.84" x2="152.4" y2="116.84" width="0.1524" layer="91"/>
-<label x="152.4" y="116.84" size="1.778" layer="95" rot="R180"/>
-</segment>
-</net>
-<net name="USB-5V-MAG" class="0">
-<segment>
-<pinref part="J1" gate="G$1" pin="VBUS"/>
-<wire x1="76.2" y1="154.94" x2="73.66" y2="154.94" width="0.1524" layer="91"/>
-<label x="73.66" y="154.94" size="1.778" layer="95" rot="R180"/>
-</segment>
-<segment>
-<pinref part="J3-M-DATA" gate="G$1" pin="VBUS"/>
-<wire x1="154.94" y1="119.38" x2="152.4" y2="119.38" width="0.1524" layer="91"/>
-<label x="152.4" y="119.38" size="1.778" layer="95" rot="R180"/>
-</segment>
-</net>
-<net name="STA-D+" class="0">
-<segment>
-<pinref part="J2" gate="G$1" pin="D+"/>
-<wire x1="76.2" y1="124.46" x2="73.66" y2="124.46" width="0.1524" layer="91"/>
-<label x="73.66" y="124.46" size="1.778" layer="95" rot="R180"/>
-</segment>
-<segment>
-<pinref part="J5-S-DATA" gate="G$1" pin="D+"/>
-<wire x1="154.94" y1="78.74" x2="152.4" y2="78.74" width="0.1524" layer="91"/>
-<label x="152.4" y="78.74" size="1.778" layer="95" rot="R180"/>
-</segment>
-</net>
-<net name="STA-D-" class="0">
-<segment>
-<pinref part="J2" gate="G$1" pin="D-"/>
-<wire x1="76.2" y1="127" x2="73.66" y2="127" width="0.1524" layer="91"/>
-<label x="73.66" y="127" size="1.778" layer="95" rot="R180"/>
-</segment>
-<segment>
-<pinref part="J5-S-DATA" gate="G$1" pin="D-"/>
-<wire x1="154.94" y1="81.28" x2="152.4" y2="81.28" width="0.1524" layer="91"/>
-<label x="152.4" y="81.28" size="1.778" layer="95" rot="R180"/>
-</segment>
-</net>
-<net name="USB-5V-STA" class="0">
-<segment>
-<pinref part="J2" gate="G$1" pin="VBUS"/>
-<wire x1="76.2" y1="129.54" x2="73.66" y2="129.54" width="0.1524" layer="91"/>
-<label x="73.66" y="129.54" size="1.778" layer="95" rot="R180"/>
-</segment>
-<segment>
-<pinref part="J5-S-DATA" gate="G$1" pin="VBUS"/>
-<wire x1="154.94" y1="83.82" x2="152.4" y2="83.82" width="0.1524" layer="91"/>
-<label x="152.4" y="83.82" size="1.778" layer="95" rot="R180"/>
-</segment>
-</net>
-<net name="USB-5V-LID" class="0">
-<segment>
-<pinref part="J8" gate="G$1" pin="VBUS"/>
-<wire x1="30.48" y1="154.94" x2="25.4" y2="154.94" width="0.1524" layer="91"/>
-<label x="25.4" y="154.94" size="1.778" layer="95" rot="R180"/>
-</segment>
-<segment>
-<pinref part="J1-L-DATA" gate="G$1" pin="VBUS"/>
-<wire x1="154.94" y1="157.48" x2="152.4" y2="157.48" width="0.1524" layer="91"/>
-<label x="152.4" y="157.48" size="1.778" layer="95" rot="R180"/>
-</segment>
-</net>
-<net name="N$2" class="0">
-<segment>
-<pinref part="J3" gate="G$1" pin="2"/>
-<pinref part="TP1" gate="G$1" pin="TP"/>
-<wire x1="60.96" y1="50.8" x2="68.58" y2="50.8" width="0.1524" layer="91"/>
-</segment>
-</net>
-<net name="N$3" class="0">
-<segment>
-<pinref part="J3" gate="G$1" pin="4"/>
-<pinref part="TP2" gate="G$1" pin="TP"/>
-<wire x1="60.96" y1="48.26" x2="71.12" y2="48.26" width="0.1524" layer="91"/>
-</segment>
-</net>
-<net name="N$4" class="0">
-<segment>
-<pinref part="J3" gate="G$1" pin="6"/>
-<pinref part="TP3" gate="G$1" pin="TP"/>
-<wire x1="60.96" y1="45.72" x2="73.66" y2="45.72" width="0.1524" layer="91"/>
-</segment>
-</net>
+</net>

Commit message: Added BOMs
Parts:
- added H1, H2, H3: MOUNT-HOLE3.0, holes:MOUNT-HOLE3.0
Changed lines of the file:
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@@
 <part name="TP2" library="testpad" library_urn="urn:adsk.eagle:library:385" deviceset="TP" device="PAD1-17" package3d_urn="urn:adsk.eagle:package:27949/1"/>
 <part name="TP3" library="testpad" library_urn="urn:adsk.eagle:library:385" deviceset="TP" device="PAD1-17" package3d_urn="urn:adsk.eagle:package:27949/1"/>
+<part name="H1" library="holes" library_urn="urn:adsk.eagle:library:237" deviceset="MOUNT-HOLE" device="3.0" package3d_urn="urn:adsk.eagle:package:14277/1"/>
+<part name="H2" library="holes" library_urn="urn:adsk.eagle:library:237" deviceset="MOUNT-HOLE" device="3.0" package3d_urn="urn:adsk.eagle:package:14277/1"/>
+<part name="H3" library="holes" library_urn="urn:adsk.eagle:library:237" deviceset="MOUNT-HOLE" device="3.0" package3d_urn="urn:adsk.eagle:package:14277/1"/>
 </parts>
 <sheets>
@@
 <attribute name="TP_SIGNAL_NAME" x="74.93" y="46.99" size="1.778" layer="97"/>
 </instance>
+<instance part="H1" gate="G$1" x="231.14" y="50.8" smashed="yes">
+<attribute name="NAME" x="233.172" y="51.3842" size="1.778" layer="95"/>
+<attribute name="VALUE" x="233.172" y="48.3362" size="1.778" layer="96"/>
+</instance>
+<instance part="H2" gate="G$1" x="231.14" y="45.72" smashed="yes">
+<attribute name="NAME" x="233.172" y="46.3042" size="1.778" layer="95"/>
+<attribute name="VALUE" x="233.172" y="43.2562" size="1.778" layer="96"/>
+</instance>
+<instance part="H3" gate="G$1" x="231.14" y="40.64" smashed="yes">
+<attribute name="NAME" x="233.172" y="41.2242" size="1.778" layer="95"/>
+<attribute name="VALUE" x="233.172" y="38.1762" size="1.778" layer="96"/>
+</instance>
 </instances>

Commit message: Finished RPi board rev 2.
Other:
- moved on the sheet: J1, J1-L-DATA, J2, J2-L-PWR, J3-M-DATA, J4-M-PWR, J5-S-DATA, J6-S-PWR, J8
Changed lines of the file:
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@@
 <layer number="115" name="ReferenceISLANDS" color="7" fill="1" visible="yes" active="yes"/>
 <layer number="116" name="Patch_BOT" color="9" fill="4" visible="yes" active="yes"/>
+<layer number="117" name="BACKMAAT1" color="7" fill="1" visible="no" active="no"/>
 <layer number="118" name="Rect_Pads" color="7" fill="1" visible="yes" active="yes"/>
+<layer number="119" name="KAP_TEKEN" color="7" fill="1" visible="no" active="no"/>
+<layer number="120" name="KAP_MAAT1" color="7" fill="1" visible="no" active="no"/>
 <layer number="121" name="_tsilk" color="7" fill="1" visible="yes" active="yes"/>
 <layer number="122" name="_bsilk" color="7" fill="1" visible="yes" active="yes"/>
@@
 <layer number="128" name="_bValues" color="7" fill="1" visible="yes" active="yes"/>
 <layer number="129" name="Mask" color="7" fill="1" visible="yes" active="yes"/>
+<layer number="130" name="SMDSTROOK" color="7" fill="1" visible="no" active="no"/>
 <layer number="131" name="tAdjust" color="7" fill="1" visible="yes" active="yes"/>
 <layer number="132" name="bAdjust" color="7" fill="1" visible="yes" active="yes"/>
+<layer number="133" name="bottom_silk" color="7" fill="1" visible="no" active="no"/>
 <layer number="144" name="Drill_legend" color="7" fill="1" visible="yes" active="yes"/>
 <layer number="150" name="Notes" color="7" fill="1" visible="yes" active="yes"/>
