File: DataControlBoard/DataControlBoard-Teensy/DataControlBoard-Teensy.sch (EAGLE design)
At the start: 61 parts, among them IC1 74LS165D, IC2 74LS165D, IC3 74AHC1G04DCK, J1 RS-Interface, J10 Magnet RPi, J11 Boom Cam RPi, J2 Pwr-Conn, J9 Static RPi, U1 MAX3232, U2 3V3REG

Commit message: Added mounting holes and rounded corners
Parts:
- added H1, H2, H3, H4, H5: MOUNT-HOLE3.2, holes:MOUNT-HOLE3.2
- added J3: Antenna SPI, SparkFun-Connectors:CONN_05LOCK
Connections:
- removed net N$30: J2.P18
- removed net N$31: J2.P19
- net ANT-MISO: now also J3.4
- net ANT-MOSI: now also J3.3
- net ANT-SCK: now also J3.5
- net ANT-SS: now also J3.1
Changed lines of the file:
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@@
 <part name="TP19" library="testpad" library_urn="urn:adsk.eagle:library:385" deviceset="TP" device="PAD1-13" package3d_urn="urn:adsk.eagle:package:27946/1"/>
 <part name="TP20" library="testpad" library_urn="urn:adsk.eagle:library:385" deviceset="TP" device="PAD1-13" package3d_urn="urn:adsk.eagle:package:27946/1"/>
+<part name="J3" library="SparkFun-Connectors" library_urn="urn:adsk.eagle:library:513" deviceset="CONN_05" device="LOCK" package3d_urn="urn:adsk.eagle:package:38105/1" value="Antenna SPI"/>
+<part name="H1" library="holes" library_urn="urn:adsk.eagle:library:237" deviceset="MOUNT-HOLE" device="3.2" package3d_urn="urn:adsk.eagle:package:14275/1"/>
+<part name="H2" library="holes" library_urn="urn:adsk.eagle:library:237" deviceset="MOUNT-HOLE" device="3.2" package3d_urn="urn:adsk.eagle:package:14275/1"/>
+<part name="H3" library="holes" library_urn="urn:adsk.eagle:library:237" deviceset="MOUNT-HOLE" device="3.2" package3d_urn="urn:adsk.eagle:package:14275/1"/>
+<part name="H4" library="holes" library_urn="urn:adsk.eagle:library:237" deviceset="MOUNT-HOLE" device="3.2" package3d_urn="urn:adsk.eagle:package:14275/1"/>
+<part name="H5" library="holes" library_urn="urn:adsk.eagle:library:237" deviceset="MOUNT-HOLE" device="3.2" package3d_urn="urn:adsk.eagle:package:14275/1"/>
 </parts>
 <sheets>
@@
 <wire x1="139.7" y1="154.94" x2="142.24" y2="154.94" width="0.1524" layer="91"/>
 <label x="142.24" y="154.94" size="1.778" layer="95" align="center-left"/>
-</segment>
-</net>
-<net name="N$30" class="0">
-<segment>
-<pinref part="J2" gate="G$1" pin="P18"/>
-<wire x1="139.7" y1="152.4" x2="142.24" y2="152.4" width="0.1524" layer="91"/>
-</segment>
-</net>
-<net name="N$31" class="0">
-<segment>
-<pinref part="J2" gate="G$1" pin="P19"/>
-<wire x1="139.7" y1="149.86" x2="142.24" y2="149.86" width="0.1524" layer="91"/>
 </segment>
 </net>
@@
 <attribute name="TP_SIGNAL_NAME" x="123.19" y="146.05" size="1.778" layer="97"/>
 </instance>
+<instance part="J3" gate="G$1" x="157.48" y="127" smashed="yes" rot="R180">
+<attribute name="VALUE" x="162.56" y="136.906" size="1.778" layer="96" font="vector" rot="R180"/>
+<attribute name="NAME" x="162.56" y="116.332" size="1.778" layer="95" font="vector" rot="R180"/>
+</instance>
+<instance part="H1" gate="G$1" x="101.6" y="10.16" smashed="yes">
+<attribute name="NAME" x="103.632" y="10.7442" size="1.778" layer="95"/>
+<attribute name="VALUE" x="103.632" y="7.6962" size="1.778" layer="96"/>
+</instance>
+<instance part="H2" gate="G$1" x="101.6" y="15.24" smashed="yes">
+<attribute name="NAME" x="103.632" y="15.8242" size="1.778" layer="95"/>
+<attribute name="VALUE" x="103.632" y="12.7762" size="1.778" layer="96"/>
+</instance>
+<instance part="H3" gate="G$1" x="101.6" y="20.32" smashed="yes">
+<attribute name="NAME" x="103.632" y="20.9042" size="1.778" layer="95"/>
+<attribute name="VALUE" x="103.632" y="17.8562" size="1.778" layer="96"/>
+</instance>
+<instance part="H4" gate="G$1" x="101.6" y="25.4" smashed="yes">
+<attribute name="NAME" x="103.632" y="25.9842" size="1.778" layer="95"/>
+<attribute name="VALUE" x="103.632" y="22.9362" size="1.778" layer="96"/>
+</instance>
+<instance part="H5" gate="G$1" x="101.6" y="30.48" smashed="yes">
+<attribute name="NAME" x="103.632" y="31.0642" size="1.778" layer="95"/>
+<attribute name="VALUE" x="103.632" y="28.0162" size="1.778" layer="96"/>
+</instance>
 </instances>
 <busses>
@@
 </segment>
 </net>
+<net name="ANT-SS" class="0">
+<segment>
+<pinref part="J3" gate="G$1" pin="1"/>
+<label x="147.32" y="132.08" size="1.778" layer="95" rot="R180"/>
+<wire x1="149.86" y1="132.08" x2="147.32" y2="132.08" width="0.1524" layer="91"/>
+</segment>
+</net>
+<net name="ANT-MOSI" class="0">
+<segment>
+<pinref part="J3" gate="G$1" pin="3"/>
+<label x="147.32" y="127" size="1.778" layer="95" rot="R180"/>
+<wire x1="149.86" y1="127" x2="147.32" y2="127" width="0.1524" layer="91"/>
+</segment>
+</net>
+<net name="ANT-MISO" class="0">
+<segment>
+<pinref part="J3" gate="G$1" pin="4"/>
+<label x="147.32" y="124.46" size="1.778" layer="95" rot="R180"/>
+<wire x1="149.86" y1="124.46" x2="147.32" y2="124.46" width="0.1524" layer="91"/>
+</segment>
+</net>
+<net name="ANT-SCK" class="0">
+<segment>
+<pinref part="J3" gate="G$1" pin="5"/>
+<label x="147.32" y="121.92" size="1.778" layer="95" rot="R180"/>
+<wire x1="149.86" y1="121.92" x2="147.32" y2="121.92" width="0.1524" layer="91"/>
+</segment>
+</net>

Commit message: added note about MSB/LSB
Other:
- note added: "PDB1 - MSB PDB16 - LSB Mines was assigned the MSB side"
Changed lines of the file:
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@@
 <text x="167.64" y="35.56" size="1.778" layer="97" rot="R90" align="top-left">Level Shift
 from 5V to 3.3V</text>
+<text x="7.62" y="116.84" size="1.778" layer="97">PDB1 - MSB
+PDB16 - LSB
+Mines was assigned the MSB side</text>
 </plain>
 <instances>

Commit message: Added rev2 , including Teensy supply voltage and other minor issues.
Parts:
- added JP1, JP2: JUMPER-SMT_2_NO_NO-SILK, SparkFun-Jumpers:JUMPER-SMT_2_NO_NO-SILK
Connections:
- removed net +3.3V: TP6.TP
- new net 3V3-JUMPERED: B1.3.3V, JP2.2
- new net 5V-JUMPERED: B1.VIN, JP1.2
- net +3V3: now also JP2.1, TP6.TP; no longer B1.3.3V
- net +5V: now also JP1.1
Changed lines of the file:
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@@
 <part name="H4" library="holes" library_urn="urn:adsk.eagle:library:237" deviceset="MOUNT-HOLE" device="3.2" package3d_urn="urn:adsk.eagle:package:14275/1"/>
 <part name="H5" library="holes" library_urn="urn:adsk.eagle:library:237" deviceset="MOUNT-HOLE" device="3.2" package3d_urn="urn:adsk.eagle:package:14275/1"/>
+<part name="JP1" library="SparkFun-Jumpers" library_urn="urn:adsk.eagle:library:528" deviceset="JUMPER-SMT_2_NO" device="_NO-SILK" package3d_urn="urn:adsk.eagle:package:39277/1"/>
+<part name="JP2" library="SparkFun-Jumpers" library_urn="urn:adsk.eagle:library:528" deviceset="JUMPER-SMT_2_NO" device="_NO-SILK" package3d_urn="urn:adsk.eagle:package:39277/1"/>
+<part name="P+2" library="supply1" library_urn="urn:adsk.eagle:library:371" deviceset="+5V" device=""/>
 </parts>
 <sheets>
@@
 <attribute name="VALUE" x="190.5" y="170.18" size="1.778" layer="96"/>
 </instance>
-<instance part="+3V3" gate="G$1" x="15.24" y="73.66" smashed="yes">
-<attribute name="VALUE" x="12.7" y="68.58" size="1.778" layer="96" rot="R90"/>
+<instance part="+3V3" gate="G$1" x="15.24" y="17.78" smashed="yes">
+<attribute name="VALUE" x="12.7" y="12.7" size="1.778" layer="96" rot="R90"/>
 </instance>
 <instance part="GND4" gate="1" x="12.7" y="45.72" smashed="yes">
@@
 <instance part="TP20" gate="G$1" x="63.5" y="76.2" smashed="yes" rot="R270">
 <attribute name="TP_SIGNAL_NAME" x="62.23" y="74.93" size="1.778" layer="97" rot="R270"/>
+</instance>
+<instance part="JP1" gate="G$1" x="22.86" y="22.86" smashed="yes">
+<attribute name="NAME" x="20.32" y="25.4" size="1.778" layer="95" font="vector"/>
+</instance>
+<instance part="JP2" gate="G$1" x="22.86" y="15.24" smashed="yes">
+<attribute name="NAME" x="20.32" y="17.78" size="1.778" layer="95" font="vector"/>
+</instance>
+<instance part="P+2" gate="1" x="15.24" y="25.4" smashed="yes">
+<attribute name="VALUE" x="15.24" y="25.4" size="1.778" layer="96"/>
 </instance>
 </instances>
@@
 </segment>
 <segment>
-<pinref part="B1" gate="G$1" pin="3.3V"/>
-<wire x1="20.32" y1="68.58" x2="15.24" y2="68.58" width="0.1524" layer="91"/>
-<wire x1="15.24" y1="68.58" x2="15.24" y2="71.12" width="0.1524" layer="91"/>
-<pinref part="+3V3" gate="G$1" pin="+3V3"/>
-</segment>
-<segment>
 <wire x1="111.76" y1="99.06" x2="111.76" y2="101.6" width="0.1524" layer="91"/>
 <pinref part="+3V7" gate="G$1" pin="+3V3"/>
@@
 <pinref part="+3V8" gate="G$1" pin="+3V3"/>
 <pinref part="IC3" gate="P" pin="VCC"/>
+</segment>
+<segment>
+<pinref part="+3V3" gate="G$1" pin="+3V3"/>
+<pinref part="JP2" gate="G$1" pin="1"/>
+<wire x1="15.24" y1="15.24" x2="17.78" y2="15.24" width="0.1524" layer="91"/>
 </segment>
 </net>
@@
 <junction x="190.5" y="162.56"/>
 </segment>
+<segment>
+<pinref part="P+2" gate="1" pin="+5V"/>
+<pinref part="JP1" gate="G$1" pin="1"/>
+<wire x1="15.24" y1="22.86" x2="17.78" y2="22.86" width="0.1524" layer="91"/>
+</segment>
 </net>
 <net name="PI-SCL" class="0">
@@
 <pinref part="B1" gate="G$1" pin="7/RX3"/>
 <wire x1="60.96" y1="76.2" x2="53.34" y2="76.2" width="0.1524" layer="91"/>
+</segment>
+</net>
+<net name="5V-JUMPERED" class="0">
+<segment>
+<pinref part="JP1" gate="G$1" pin="2"/>
+<wire x1="27.94" y1="22.86" x2="30.48" y2="22.86" width="0.1524" layer="91"/>
+<label x="30.48" y="22.86" size="1.27" layer="95" xref="yes"/>
+</segment>
+<segment>
+<pinref part="B1" gate="G$1" pin="VIN"/>
+<wire x1="20.32" y1="73.66" x2="17.78" y2="73.66" width="0.1524" layer="91"/>
+<label x="17.78" y="73.66" size="1.27" layer="95" rot="R180" xref="yes"/>
+</segment>
+</net>
+<net name="3V3-JUMPERED" class="0">
+<segment>
+<pinref part="JP2" gate="G$1" pin="2"/>
+<wire x1="27.94" y1="15.24" x2="30.48" y2="15.24" width="0.1524" layer="91"/>
+<label x="30.48" y="15.24" size="1.27" layer="95" xref="yes"/>
+</segment>
+<segment>
+<pinref part="B1" gate="G$1" pin="3.3V"/>
+<wire x1="20.32" y1="68.58" x2="17.78" y2="68.58" width="0.1524" layer="91"/>
+<label x="17.78" y="68.58" size="1.27" layer="95" rot="R180" xref="yes"/>
 </segment>
 </net>
@@
 <junction x="40.64" y="154.94"/>
 </segment>
+<segment>
+<pinref part="TP6" gate="G$1" pin="TP"/>
+<wire x1="111.76" y1="149.86" x2="109.22" y2="149.86" width="0.1524" layer="91"/>
+<label x="109.22" y="149.86" size="1.778" layer="95" rot="R180"/>
+</segment>
 </net>
 <net name="SDA0" class="0">
@@
 </segment>
 </net>
-<net name="+3.3V" class="0">
-<segment>
-<pinref part="TP6" gate="G$1" pin="TP"/>
-<wire x1="111.76" y1="149.86" x2="109.22" y2="149.86" width="0.1524" layer="91"/>
-<label x="109.22" y="149.86" size="1.778" layer="95" rot="R180"/>
-</segment>
-</net>

Commit message: Moved some files around. Made progress on power management board
Connections:
- new net ANT-BUSY: J3.2
- new net CAM-USB_N: J2.P19
- new net CAM-USB_P: J2.P18
Changed lines of the file:
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@@
-</segment>
-</net>
-<net name="ANT-SS" class="0">
-<segment>
-<pinref part="J2" gate="G$1" pin="P17"/>
-<wire x1="139.7" y1="154.94" x2="142.24" y2="154.94" width="0.1524" layer="91"/>
-<label x="142.24" y="154.94" size="1.778" layer="95" align="center-left"/>
 </segment>
 </net>
@@
 <wire x1="20.32" y1="68.58" x2="17.78" y2="68.58" width="0.1524" layer="91"/>
 <label x="17.78" y="68.58" size="1.27" layer="95" rot="R180" xref="yes"/>
+</segment>
+</net>
+<net name="ANT-SS" class="0">
+<segment>
+<pinref part="J2" gate="G$1" pin="P17"/>
+<wire x1="139.7" y1="154.94" x2="142.24" y2="154.94" width="0.1524" layer="91"/>
+<label x="142.24" y="154.94" size="1.778" layer="95" align="center-left"/>
+</segment>
+</net>
+<net name="CAM-USB_P" class="0">
+<segment>
+<pinref part="J2" gate="G$1" pin="P18"/>
+<wire x1="139.7" y1="152.4" x2="142.24" y2="152.4" width="0.1524" layer="91"/>
+<label x="142.24" y="152.4" size="1.778" layer="95"/>
+</segment>
+</net>
+<net name="CAM-USB_N" class="0">
+<segment>
+<pinref part="J2" gate="G$1" pin="P19"/>
+<wire x1="139.7" y1="149.86" x2="142.24" y2="149.86" width="0.1524" layer="91"/>
+<label x="142.24" y="149.86" size="1.778" layer="95"/>
 </segment>
 </net>
@@
 <segment>
 <pinref part="J3" gate="G$1" pin="1"/>
-<label x="147.32" y="132.08" size="1.778" layer="95" rot="R180"/>
+<label x="147.32" y="132.08" size="1.27" layer="95" rot="R180" xref="yes"/>
 <wire x1="149.86" y1="132.08" x2="147.32" y2="132.08" width="0.1524" layer="91"/>
 </segment>
@@
 <segment>
 <pinref part="J3" gate="G$1" pin="3"/>
-<label x="147.32" y="127" size="1.778" layer="95" rot="R180"/>
+<label x="147.32" y="127" size="1.27" layer="95" rot="R180" xref="yes"/>
 <wire x1="149.86" y1="127" x2="147.32" y2="127" width="0.1524" layer="91"/>
 </segment>
@@
 <segment>
 <pinref part="J3" gate="G$1" pin="4"/>
-<label x="147.32" y="124.46" size="1.778" layer="95" rot="R180"/>
+<label x="147.32" y="124.46" size="1.27" layer="95" rot="R180" xref="yes"/>
 <wire x1="149.86" y1="124.46" x2="147.32" y2="124.46" width="0.1524" layer="91"/>
 </segment>
@@
 <segment>
 <pinref part="J3" gate="G$1" pin="5"/>
-<label x="147.32" y="121.92" size="1.778" layer="95" rot="R180"/>
+<label x="147.32" y="121.92" size="1.27" layer="95" rot="R180" xref="yes"/>
 <wire x1="149.86" y1="121.92" x2="147.32" y2="121.92" width="0.1524" layer="91"/>
 </segment>
 </net>
+<net name="ANT-BUSY" class="0">
+<segment>
+<pinref part="J3" gate="G$1" pin="2"/>
+<wire x1="149.86" y1="129.54" x2="147.32" y2="129.54" width="0.1524" layer="91"/>
+<label x="147.32" y="129.54" size="1.27" layer="95" rot="R180" xref="yes"/>
+</segment>
+</net>

Commit message: Implemented ANT-BUSY signal to replace 5V supply on lidar
Parts:
- added TP21: TPPAD1-13, testpad:TPPAD1-13
Connections:
- net ANT-BUSY: now also J2.P3
- net LASER-VS-1: now also TP21.TP; no longer J2.P3

Commit message: Routed data control board
Parts:
- added TP22, TP23: TPPAD1-13, testpad:TPPAD1-13
Connections:
- net CAM-USB_N: now also TP23.TP
- net CAM-USB_P: now also TP22.TP
Changed lines of the file:
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@@
 <class number="0" name="default" width="0" drill="0">
+</class>
+<class number="1" name="USB-Diff" width="0.254" drill="0">
+<clearance class="0" value="0.3048"/>
+<clearance class="1" value="0.1524"/>
 </class>
 </classes>
@@
 <part name="P+2" library="supply1" library_urn="urn:adsk.eagle:library:371" deviceset="+5V" device=""/>
 <part name="TP21" library="testpad" library_urn="urn:adsk.eagle:library:385" deviceset="TP" device="PAD1-13" package3d_urn="urn:adsk.eagle:package:27946/1"/>
+<part name="TP22" library="testpad" library_urn="urn:adsk.eagle:library:385" deviceset="TP" device="PAD1-13" package3d_urn="urn:adsk.eagle:package:27946/1" value="TPPAD1-13"/>
+<part name="TP23" library="testpad" library_urn="urn:adsk.eagle:library:385" deviceset="TP" device="PAD1-13" package3d_urn="urn:adsk.eagle:package:27946/1" value="TPPAD1-13"/>
 </parts>
 <sheets>
@@
 </segment>
 </net>
-<net name="CAM-USB_P" class="0">
+<net name="CAM-USB_P" class="1">
 <segment>
 <pinref part="J2" gate="G$1" pin="P18"/>
@@
 </segment>
 </net>
-<net name="CAM-USB_N" class="0">
+<net name="CAM-USB_N" class="1">
 <segment>
 <pinref part="J2" gate="G$1" pin="P19"/>
@@
 <attribute name="TP_SIGNAL_NAME" x="158.75" y="54.61" size="1.778" layer="97"/>
 </instance>
+<instance part="TP22" gate="G$1" x="127" y="101.6" smashed="yes">
+<attribute name="NAME" x="125.73" y="102.87" size="1.778" layer="95"/>
+<attribute name="TP_SIGNAL_NAME" x="128.27" y="100.33" size="1.778" layer="97"/>
+</instance>
+<instance part="TP23" gate="G$1" x="129.54" y="96.52" smashed="yes">
+<attribute name="NAME" x="128.27" y="97.79" size="1.778" layer="95"/>
+<attribute name="TP_SIGNAL_NAME" x="130.81" y="95.25" size="1.778" layer="97"/>
+</instance>
 </instances>
 <busses>
@@
 </segment>
 </net>
+<net name="CAM-USB_P" class="1">
+<segment>
+<pinref part="TP22" gate="G$1" pin="TP"/>
+<wire x1="127" y1="99.06" x2="124.46" y2="99.06" width="0.1524" layer="91"/>
+<label x="124.46" y="99.06" size="1.27" layer="95" rot="R180" xref="yes"/>
+</segment>
+</net>
+<net name="CAM-USB_N" class="1">
+<segment>
+<pinref part="TP23" gate="G$1" pin="TP"/>
+<wire x1="129.54" y1="93.98" x2="124.46" y2="93.98" width="0.1524" layer="91"/>
+<label x="124.46" y="93.98" size="1.27" layer="95" rot="R180" xref="yes"/>
+</segment>
+</net>
