File: microDB-Breakout/board.brd (EAGLE design)
At the start: 8.9 x 20.3 mm, 26 parts, among them P1 TP-19MIL, P10 TP-19MIL, P11 TP-19MIL, P12 TP-19MIL, P13 TP-19MIL, P14 TP-19MIL, P15 TP-19MIL, P16 TP-19MIL, P17 TP-19MIL, P18 TP-19MIL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

Commit message: Partially Routed
Parts:
- moved P16 51.6 mm to (10.5, 16.5)
- moved P17 51.6 mm to (10.5, 14.0)
- moved P18 47.3 mm to (6.99, 7.62)
- moved P19 47.3 mm to (6.99, 5.08)
- moved P21 43.6 mm to (7.62, -1.27)
- moved P20 43.3 mm to (7.62, 1.27), turned to 180 degrees
- moved P23 41.1 mm to (7.62, -6.35)
- moved P24 41.1 mm to (7.62, -8.89)
- moved P22 40.8 mm to (7.62, -3.81)
- moved P25 38.3 mm to (7.62, -11.4)
- moved P3 25.8 mm to (10.5, 17.8)
- moved P4 25.8 mm to (10.5, 15.2)
- moved P5 21.1 mm to (6.99, 8.89)
- moved P6 21.1 mm to (6.99, 6.35)
- moved P7 21.1 mm to (6.99, 3.81)
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Routing:
- net N$3: track 0.00 -> 14.5 mm
- net N$16: track 0.00 -> 12.5 mm
- net N$15: track 0.00 -> 11.8 mm
- net N$2: track 0.00 -> 11.2 mm
- net N$1: track 0.00 -> 7.34 mm
- net N$14: track 0.00 -> 5.36 mm
Other:
- board size 8.9 x 20.3 mm -> 14.6 x 20.3 mm
